File: Keyboard PCB/Keyboard PCB.kicad_pcb (KiCad board)
At the start: 2 copper layers, 25 parts, among them J1 USB_B_Mini, SW1 SW_Push, SW2 MXSwitch, SW3 MXSwitch, SW4 MXSwitch, SW5 MXSwitch, U1 ATmega32U4-AU, Y1 16mhz

Commit message: ROW2
Parts:
- U1: footprint Package_QFP:TQFP-44_10x10mm_P0.8mm -> acheron_Components:TQPF-44_10x10mm_P0.8mm
- Y1: footprint Crystal:Crystal_SMD_5032-2Pin_5.0x3.2mm_HandSoldering -> Crystal:Crystal_SMD_3225-4Pin_3.2x2.5mm_HandSoldering
- moved C2 70.1 mm to (308.4, -31.6)
- moved D2 54.9 mm to (308.8, -34.8)
- moved C6 40.3 mm to (314.1, -34.9)
- moved C4 34.0 mm to (292.2, -17.2)
- moved Y1 28.5 mm to (298.2, -22.1)
- moved SW5 23.7 mm to (284.0, -18.6)
- moved C3 20.7 mm to (287.4, -10.7)
- moved D3 20.0 mm to (282.1, -13.6)
- moved U1 19.5 mm to (287.6, -29.2)
- moved J1 19.4 mm to (300.4, -34.0)
- moved C1 19.3 mm to (297.2, -17.8)
- moved R4 19.1 mm to (259.8, 5.49)
- moved R1 19.1 mm to (241.9, 5.49)
- moved R2 19.1 mm to (247.9, 5.49)
- moved R3 19.1 mm to (253.8, 5.49)
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
Commit message: switches placed
Parts:
- added D10: 1N4148W, Diode_SMD:D_SOD-123, B.Cu at (-34.9, -156.5)
- added D11: 1N4148W, Diode_SMD:D_SOD-123, B.Cu at (-29.1, -156.5)
- added D12: 1N4148W, Diode_SMD:D_SOD-123, B.Cu at (-23.4, -156.5)
- added D13: 1N4148W, Diode_SMD:D_SOD-123, B.Cu at (-17.6, -156.5)
- added D14: 1N4148W, Diode_SMD:D_SOD-123, B.Cu at (11.1, -184.7)
- added D15: 1N4148W, Diode_SMD:D_SOD-123, B.Cu at (-6.10, -156.5)
- added D16: 1N4148W, Diode_SMD:D_SOD-123, B.Cu at (-63.6, -158.4)
- added D17: 1N4148W, Diode_SMD:D_SOD-123, B.Cu at (5.40, -156.5)
- added D18: 1N4148W, Diode_SMD:D_SOD-123, B.Cu at (11.2, -156.3)
- added D19: 1N4148W, Diode_SMD:D_SOD-123, B.Cu at (16.9, -156.3)
- added D20: 1N4148W, Diode_SMD:D_SOD-123, B.Cu at (11.2, -159.7)
- added D21: 1N4148W, Diode_SMD:D_SOD-123, B.Cu at (16.9, -159.7)
- added D22: 1N4148W, Diode_SMD:D_SOD-123, B.Cu at (22.6, -157.8)
- added D23: 1N4148W, Diode_SMD:D_SOD-123, B.Cu at (-75.1, -247.9)
- added D24: 1N4148W, Diode_SMD:D_SOD-123, B.Cu at (-75.1, -251.3)
- added D25: 1N4148W, Diode_SMD:D_SOD-123, B.Cu at (-11.8, -156.5)
- added D26: 1N4148W, Diode_SMD:D_SOD-123, B.Cu at (-69.3, -251.3)
- added D27: 1N4148W, Diode_SMD:D_SOD-123, B.Cu at (34.1, -157.8)
- added D28: 1N4148W, Diode_SMD:D_SOD-123, B.Cu at (39.9, -157.8)
- added D29: 1N4148W, Diode_SMD:D_SOD-123, B.Cu at (45.6, -157.8)
- added D30: 1N4148W, Diode_SMD:D_SOD-123, B.Cu at (16.9, -184.7)
- added D31: 1N4148W, Diode_SMD:D_SOD-123, B.Cu at (11.1, -188.0)
- added D32: 1N4148W, Diode_SMD:D_SOD-123, B.Cu at (11.1, -191.4)
- added D33: 1N4148W, Diode_SMD:D_SOD-123, B.Cu at (11.1, -194.7)
- added D34: 1N4148W, Diode_SMD:D_SOD-123, B.Cu at (16.9, -188.0)
- added D35: 1N4148W, Diode_SMD:D_SOD-123, B.Cu at (-69.3, -247.9)
- added D36: 1N4148W, Diode_SMD:D_SOD-123, B.Cu at (-63.6, -261.3)
- added D37: 1N4148W, Diode_SMD:D_SOD-123, B.Cu at (28.4, -157.8)
- added D38: 1N4148W, Diode_SMD:D_SOD-123, B.Cu at (-63.6, -251.3)
- added D39: 1N4148W, Diode_SMD:D_SOD-123, B.Cu at (-75.1, -254.6)
- added D40: 1N4148W, Diode_SMD:D_SOD-123, B.Cu at (-75.1, -258.0)
- added D41: 1N4148W, Diode_SMD:D_SOD-123, B.Cu at (-75.1, -261.3)
- added D42: 1N4148W, Diode_SMD:D_SOD-123, B.Cu at (-69.3, -254.6)
- added D43: 1N4148W, Diode_SMD:D_SOD-123, B.Cu at (-63.6, -254.6)
- added D44: 1N4148W, Diode_SMD:D_SOD-123, B.Cu at (-69.3, -258.0)
- added D45: 1N4148W, Diode_SMD:D_SOD-123, B.Cu at (-63.6, -258.0)
- added D46: 1N4148W, Diode_SMD:D_SOD-123, B.Cu at (-69.3, -261.3)
- added D47: 1N4148W, Diode_SMD:D_SOD-123, B.Cu at (-63.6, -247.9)
- added D48: 1N4148W, Diode_SMD:D_SOD-123, B.Cu at (-0.35, -156.5)
- added D49: 1N4148W, Diode_SMD:D_SOD-123, B.Cu at (22.6, -184.7)
- added D5: 1N4148W, Diode_SMD:D_SOD-123, B.Cu at (57.1, -157.8)
- added D50: 1N4148W, Diode_SMD:D_SOD-123, B.Cu at (22.6, -188.0)
- added D51: 1N4148W, Diode_SMD:D_SOD-123, B.Cu at (16.9, -191.4)
- added D52: 1N4148W, Diode_SMD:D_SOD-123, B.Cu at (22.6, -191.4)
- added D53: 1N4148W, Diode_SMD:D_SOD-123, B.Cu at (16.9, -194.7)
- added D54: 1N4148W, Diode_SMD:D_SOD-123, B.Cu at (22.6, -194.7)
- added D55: 1N4148W, Diode_SMD:D_SOD-123, B.Cu at (11.1, -198.1)
- added D56: 1N4148W, Diode_SMD:D_SOD-123, B.Cu at (16.9, -198.1)
- added D57: 1N4148W, Diode_SMD:D_SOD-123, B.Cu at (22.6, -198.1)
- added D58: 1N4148W, Diode_SMD:D_SOD-123, B.Cu at (-15.8, -239.3)
- added D59: 1N4148W, Diode_SMD:D_SOD-123, B.Cu at (51.4, -157.8)
- added D6: 1N4148W, Diode_SMD:D_SOD-123, B.Cu at (-57.9, -158.4)
- added D60: 1N4148W, Diode_SMD:D_SOD-123, B.Cu at (62.9, -157.8)
- added D61: 1N4148W, Diode_SMD:D_SOD-123, B.Cu at (-15.8, -225.9)
- added D62: 1N4148W, Diode_SMD:D_SOD-123, B.Cu at (-10.1, -225.9)
- added D63: 1N4148W, Diode_SMD:D_SOD-123, B.Cu at (-15.8, -229.2)
- added D64: 1N4148W, Diode_SMD:D_SOD-123, B.Cu at (-10.1, -229.2)
- added D65: 1N4148W, Diode_SMD:D_SOD-123, B.Cu at (-15.8, -232.6)
- added D66: 1N4148W, Diode_SMD:D_SOD-123, B.Cu at (-10.1, -232.6)
- added D67: 1N4148W, Diode_SMD:D_SOD-123, B.Cu at (-15.8, -235.9)
- added D68: 1N4148W, Diode_SMD:D_SOD-123, B.Cu at (-10.1, -235.9)
- added D69: 1N4148W, Diode_SMD:D_SOD-123, B.Cu at (59.9, -239.5)
- added D7: 1N4148W, Diode_SMD:D_SOD-123, B.Cu at (-52.1, -158.4)
- added D70: 1N4148W, Diode_SMD:D_SOD-123, B.Cu at (15.9, -225.9)
- added D71: 1N4148W, Diode_SMD:D_SOD-123, B.Cu at (15.9, -229.2)
- added D72: 1N4148W, Diode_SMD:D_SOD-123, B.Cu at (15.9, -232.6)
- added D73: 1N4148W, Diode_SMD:D_SOD-123, B.Cu at (15.9, -235.9)
- added D74: 1N4148W, Diode_SMD:D_SOD-123, B.Cu at (15.9, -239.3)
- added D75: 1N4148W, Diode_SMD:D_SOD-123, B.Cu at (48.4, -226.1)
- added D76: 1N4148W, Diode_SMD:D_SOD-123, B.Cu at (54.1, -226.1)
- added D77: 1N4148W, Diode_SMD:D_SOD-123, B.Cu at (59.9, -226.1)
- added D78: 1N4148W, Diode_SMD:D_SOD-123, B.Cu at (48.4, -229.4)
- added D79: 1N4148W, Diode_SMD:D_SOD-123, B.Cu at (54.1, -229.4)
- added D8: 1N4148W, Diode_SMD:D_SOD-123, B.Cu at (-46.4, -158.4)
- added D80: 1N4148W, Diode_SMD:D_SOD-123, B.Cu at (-10.1, -239.3)
- added D81: 1N4148W, Diode_SMD:D_SOD-123, B.Cu at (54.1, -239.5)
- added D82: 1N4148W, Diode_SMD:D_SOD-123, B.Cu at (48.4, -239.5)
- added D83: 1N4148W, Diode_SMD:D_SOD-123, B.Cu at (59.9, -236.1)
- added D84: 1N4148W, Diode_SMD:D_SOD-123, B.Cu at (54.1, -236.1)
- added D85: 1N4148W, Diode_SMD:D_SOD-123, B.Cu at (48.4, -236.1)
- added D86: 1N4148W, Diode_SMD:D_SOD-123, B.Cu at (59.9, -232.8)
- added D87: 1N4148W, Diode_SMD:D_SOD-123, B.Cu at (54.1, -232.8)
- added D88: 1N4148W, Diode_SMD:D_SOD-123, B.Cu at (48.4, -232.8)
- added D89: 1N4148W, Diode_SMD:D_SOD-123, B.Cu at (59.9, -229.4)
- added D9: 1N4148W, Diode_SMD:D_SOD-123, B.Cu at (-40.6, -158.4)
- added D90: 1N4148W, Diode_SMD:D_SOD-123, B.Cu at (100.0, -185.7)
- added SW10: F8, acheron_MX:MX100, B.Cu at (-190.5, -314.3)
- added SW11: F10, acheron_MX:MX100, B.Cu at (-190.5, -295.3)
- added SW12: ESC, acheron_MX:MX100, B.Cu at (-166.7, -371.5)
- added SW13: Tab, acheron_MX:MX150, B.Cu at (-161.9, -352.4)
- added SW14: L Shift, acheron_MX:MX225, B.Cu at (-154.8, -314.3)
- added SW15: L Ctrl, acheron_MX:MX150, B.Cu at (-161.9, -295.3)
- added SW16: 1, acheron_MX:MX100, B.Cu at (-147.6, -371.5)
- added SW17: Q, acheron_MX:MX100, B.Cu at (-138.1, -352.4)
- added SW18: A, acheron_MX:MX100, B.Cu at (-133.3, -333.4)
- added SW19: S, acheron_MX:MX100, B.Cu at (-114.3, -333.4)
- added SW20: 2, acheron_MX:MX100, B.Cu at (-128.6, -371.5)
- added SW21: W, acheron_MX:MX100, B.Cu at (-119.1, -352.4)
- added SW22: Z, acheron_MX:MX100, B.Cu at (-123.8, -314.3)
- added SW23: L Alt, acheron_MX:MX150, B.Cu at (-119.1, -295.3)
- added SW24: 3, acheron_MX:MX100, B.Cu at (-109.5, -371.5)
- added SW25: E, acheron_MX:MX100, B.Cu at (-100.0, -352.4)
- added SW26: D, acheron_MX:MX100, B.Cu at (-95.2, -333.4)
- added SW27: X, acheron_MX:MX100, B.Cu at (-104.8, -314.3)
- added SW28: 4, acheron_MX:MX100, B.Cu at (-90.5, -371.5)
- added SW29: R, acheron_MX:MX100, B.Cu at (-81.0, -352.4)
- added SW30: F, acheron_MX:MX100, B.Cu at (-76.2, -333.4)
- added SW31: C, acheron_MX:MX100, B.Cu at (-85.7, -314.3)
- added SW32: 5, acheron_MX:MX100, B.Cu at (-71.4, -371.5)
- added SW33: T, acheron_MX:MX100, B.Cu at (-61.9, -352.4)
- added SW34: G, acheron_MX:MX100, B.Cu at (-57.1, -333.4)
- added SW35: V, acheron_MX:MX100, B.Cu at (-66.7, -314.3)
- added SW36: 6, acheron_MX:MX100, B.Cu at (-52.4, -371.5)
- added SW37: Y, acheron_MX:MX100, B.Cu at (-42.9, -352.4)
- added SW38: H, acheron_MX:MX100, B.Cu at (-38.1, -333.4)
- added SW39: B, acheron_MX:MX100, B.Cu at (-47.6, -314.3)
- added SW40: Space, acheron_MX:MX625, B.Cu at (-45.2, -295.3)
- added SW41: 7, acheron_MX:MX100, B.Cu at (-33.3, -371.5)
- added SW42: U, acheron_MX:MX100, B.Cu at (-23.8, -352.4)
- added SW43: J, acheron_MX:MX100, B.Cu at (-19.1, -333.4)
- added SW44: N, acheron_MX:MX100, B.Cu at (-28.6, -314.3)
- added SW45: 8, acheron_MX:MX100, B.Cu at (-14.3, -371.5)
- added SW46: I, acheron_MX:MX100, B.Cu at (-4.76, -352.4)
- added SW47: K, acheron_MX:MX100, B.Cu at (0.00, -333.4)
- added SW48: M, acheron_MX:MX100, B.Cu at (-9.53, -314.3)
- added SW49: 9, acheron_MX:MX100, B.Cu at (4.76, -371.5)
- added SW50: O, acheron_MX:MX100, B.Cu at (14.3, -352.4)
- added SW51: L, acheron_MX:MX100, B.Cu at (19.1, -333.4)
- added SW52: ,, acheron_MX:MX100, B.Cu at (9.53, -314.3)
- added SW53: AltGr, acheron_MX:MX100, B.Cu at (23.8, -295.3)
- added SW54: ;, acheron_MX:MX100, B.Cu at (38.1, -333.4)
- added SW55: FN, acheron_MX:MX100, B.Cu at (42.9, -295.3)
- added SW56: 0, acheron_MX:MX100, B.Cu at (23.8, -371.5)
- added SW57: P, acheron_MX:MX100, B.Cu at (33.3, -352.4)
- added SW58: ., acheron_MX:MX100, B.Cu at (28.6, -314.3)
- added SW59: R Ctrl, acheron_MX:MX100, B.Cu at (61.9, -295.3)
- added SW6: F5, acheron_MX:MX100, B.Cu at (-209.6, -333.4)
- added SW60: -, acheron_MX:MX100, B.Cu at (42.9, -371.5)
- added SW61: [, acheron_MX:MX100, B.Cu at (52.4, -352.4)
- added SW62: ', acheron_MX:MX100, B.Cu at (57.1, -333.4)
- added SW63: /, acheron_MX:MX100, B.Cu at (47.6, -314.3)
- added SW64: =, acheron_MX:MX100, B.Cu at (61.9, -371.5)
- added SW65: ], acheron_MX:MX100, B.Cu at (71.4, -352.4)
- added SW66: RShift, acheron_MX:MX175, B.Cu at (73.8, -314.3)
- added SW67: Left, acheron_MX:MX100, B.Cu at (85.7, -290.5)
- added SW68: Back Space, acheron_MX:MX200, B.Cu at (90.5, -371.5)
- added SW69: \, acheron_MX:MX150, B.Cu at (95.2, -352.4)
- added SW7: F7, acheron_MX:MX100, B.Cu at (-209.6, -314.3)
- added SW70: Enter, acheron_MX:MX225, B.Cu at (88.1, -333.4)
- added SW71: UP, acheron_MX:MX100, B.Cu at (104.8, -309.6)
- added SW72: Down, acheron_MX:MX100, B.Cu at (104.8, -290.5)
- added SW73: Right, acheron_MX:MX100, B.Cu at (123.8, -290.5)
- added SW74: Num lock, acheron_MX:MX100, B.Cu at (128.6, -371.5)
- added SW75: N7, acheron_MX:MX100, B.Cu at (128.6, -352.4)
- added SW76: N1, acheron_MX:MX100, B.Cu at (128.6, -314.3)
- added SW77: N4, acheron_MX:MX100, B.Cu at (128.6, -333.4)
- added SW78: N/, acheron_MX:MX100, B.Cu at (147.6, -371.5)
- added SW79: N8, acheron_MX:MX100, B.Cu at (147.6, -352.4)
- added SW8: F9, acheron_MX:MX100, B.Cu at (-209.6, -295.3)
- added SW80: N2, acheron_MX:MX100, B.Cu at (147.6, -314.3)
- added SW81: N5, acheron_MX:MX100, B.Cu at (147.6, -333.4)
- added SW82: N0, acheron_MX:MX100, B.Cu at (147.6, -295.3)
- added SW83: N*, acheron_MX:MX100, B.Cu at (166.7, -371.5)
- added SW84: N9, acheron_MX:MX100, B.Cu at (166.7, -352.4)
- added SW85: N3, acheron_MX:MX100, B.Cu at (166.7, -314.3)
- added SW86: N6, acheron_MX:MX100, B.Cu at (166.7, -333.4)
- added SW87: N., acheron_MX:MX100, B.Cu at (166.7, -295.3)
- added SW88: N-, acheron_MX:MX100, B.Cu at (185.7, -371.5)
- added SW89: N+, acheron_MX:MX200V, B.Cu at (185.7, -342.9)
- added SW9: F6, acheron_MX:MX100, B.Cu at (-190.5, -333.4)
- added SW90: PEenter, acheron_MX:MX200V, B.Cu at (185.7, -304.8)
- added SW91: Caps, acheron_MX:MX175, B.Cu at (-159.6, -333.4)
- C1, C2, C3, C4, C5, C6, C7, C8, D1, D2, D3, D4, J1, R1, R2, R3, R4, R5, U1, Y1: moved to B.Cu
- SW1: footprint acheron_MX:MX100 -> acheron_Hardware:smdPushBtn; moved to B.Cu
- SW2: value MXSwitch -> F1; moved to B.Cu
- SW3: value MXSwitch -> F3; moved to B.Cu
- SW4: value MXSwitch -> F2; moved to B.Cu
- SW5: value MXSwitch -> F4; footprint acheron_Hardware:smdPushBtn -> acheron_MX:MX100; moved to B.Cu
- moved SW2 590.1 mm to (-209.6, -371.5), turned to 180 degrees
- moved SW5 580.2 mm to (-190.5, -352.4), turned to 180 degrees
- moved SW3 574.6 mm to (-209.6, -352.4), turned to 180 degrees
- moved SW4 558.8 mm to (-190.5, -371.5), turned to 180 degrees
- moved C6 487.8 mm to (-154.7, -169.5), turned to 180 degrees
- moved C2 478.7 mm to (-149.0, -172.9), turned to 180 degrees
- moved D2 477.7 mm to (-149.4, -169.7), turned to 180 degrees
- moved J1 472.0 mm to (-23.8, -377.1)
- moved C1 466.6 mm to (-137.8, -186.7), turned to 180 degrees
- moved Y1 465.4 mm to (-138.8, -182.3), turned to 180 degrees
- moved C4 457.8 mm to (-132.8, -187.3), turned to 180 degrees
- moved R5 454.7 mm to (-132.4, -184.1), turned to 180 degrees
- moved C3 454.0 mm to (-128.0, -193.8), turned to 180 degrees
- moved C8 451.6 mm to (-128.0, -190.7), turned to 180 degrees
- moved C5 449.2 mm to (-122.3, -200.5), turned to 180 degrees
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Connections:
- D1 pad 1: ROW2 -> ROW1
- D2 pad 1: ROW1 -> ROW2
- D3 pad 1: ROW2 -> ROW1
- D4 pad 1: ROW1 -> ROW2
Other:
- board outline added: 419.1 x 104.8 mm

Commit message: Diodes placing
Parts:
- moved D71 531.4 mm to (333.3, 197.0)
- moved D72 531.4 mm to (333.3, 193.6)
- moved D70 531.4 mm to (333.3, 200.3)
- moved D73 531.4 mm to (333.3, 190.3)
- moved D74 531.4 mm to (333.3, 186.9)
- moved D80 524.4 mm to (364.3, 127.9), turned to 90 degrees
- moved C5 520.5 mm to (235.8, 177.3), turned to 0 degrees
- moved J1 513.7 mm to (200.5, 85.0)
- moved SW10 513.7 mm to (33.8, 147.8)
- moved SW11 513.7 mm to (33.8, 166.8)
- moved SW12 513.7 mm to (57.6, 90.6)
- moved SW13 513.7 mm to (62.4, 109.7)
- moved SW14 513.7 mm to (69.5, 147.8)
- moved SW15 513.7 mm to (62.4, 166.8)
- moved SW16 513.7 mm to (76.7, 90.6)
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
Commit message: Routing
Parts:
- moved D5 283.3 mm to (7.14, 128.6), turned to 90 degrees
- moved D90 252.3 mm to (57.1, 128.6), turned to 90 degrees
- moved D14 193.6 mm to (54.8, 166.7), turned to 90 degrees
- moved D19 193.3 mm to (88.1, 90.5), turned to 90 degrees
- moved D15 190.2 mm to (69.1, 90.5), turned to 90 degrees
- moved D11 187.2 mm to (50.0, 90.5), turned to 90 degrees
- moved D27 176.7 mm to (126.2, 90.5), turned to 90 degrees
- moved D12 176.2 mm to (54.8, 109.5), turned to 90 degrees
- moved D67 173.2 mm to (307.2, 90.5), turned to 90 degrees
- moved D8 169.6 mm to (26.2, 128.6), turned to 90 degrees
- moved D6 168.2 mm to (7.14, 147.6), turned to 90 degrees
- moved D7 167.6 mm to (7.14, 166.7), turned to 90 degrees
- moved D20 167.5 mm to (97.6, 109.5), turned to 90 degrees
- moved D9 166.6 mm to (26.2, 147.6), turned to 90 degrees
- moved D10 166.4 mm to (26.2, 166.7), turned to 90 degrees
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Connections:
- SW54 pad 1: Net-(SW54-Pad1) -> COL13
- SW55 pad 1: Net-(SW54-Pad1) -> COL13
- SW58 pad 1: Net-(SW54-Pad1) -> COL13
- U1 pad 25: Net-(U1-Pad25) -> COL1
- U1 pad 26: Net-(U1-Pad26) -> COL2
- U1 pad 27: Net-(U1-Pad27) -> COL3
- U1 pad 28: Net-(U1-Pad28) -> COL4
- U1 pad 29: Net-(U1-Pad29) -> COL5
- U1 pad 30: Net-(U1-Pad30) -> COL6
- U1 pad 31: Net-(U1-Pad31) -> COL7
- U1 pad 32: Net-(U1-Pad32) -> COL8
- U1 pad 36: Net-(U1-Pad36) -> COL9
- U1 pad 37: Net-(U1-Pad37) -> COL10
- U1 pad 38: Net-(U1-Pad38) -> COL11
- U1 pad 39: Net-(U1-Pad39) -> COL12
- U1 pad 40: Net-(U1-Pad40) -> COL13
- U1 pad 41: Net-(U1-Pad41) -> COL14
Routing:
- net ROW4: track 0.00 -> 414.3 mm
- net ROW5: track 0.00 -> 322.0 mm, vias 0 -> 4
- net COL1: track 0.00 -> 264.9 mm, vias 0 -> 1
- net COL2: track 0.00 -> 245.5 mm
- net COL3: track 0.00 -> 224.6 mm
- net COL4: track 0.00 -> 199.8 mm, vias 0 -> 3
- net GND: track 0.00 -> 196.0 mm, vias 0 -> 7
- net COL5: track 0.00 -> 184.9 mm
- net COL6: track 0.00 -> 159.7 mm, vias 0 -> 1
- net COL7: track 0.00 -> 141.1 mm, vias 0 -> 1
- net COL8: track 0.00 -> 122.0 mm, vias 0 -> 1
- net +5V: track 0.00 -> 109.3 mm, vias 0 -> 1
- net COL10: track 0.00 -> 104.1 mm, vias 0 -> 6
- net COL11: track 0.00 -> 97.3 mm, vias 0 -> 4
- net Net-(R4-Pad1): track 0.00 -> 96.8 mm, vias 0 -> 2
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Other:
- net class Default: trace_width 0.25 -> 0.254
- net class Power added: clearance 0.2, trace_width 0.381, via_dia 0.8, via_drill 0.4
