File: Keyboard PCB/Keyboard PCB.sch (KiCad schematic (older format))
At the start: 195 parts, among them J1 USB_B_Mini, SW1 SW_Push, SW10 F8, SW11 F10, SW12 ESC, SW13 Tab, SW14 L Shift, SW15 L Ctrl, SW16 1, SW17 Q, SW18 A, SW19 S, SW2 F1, SW20 2, SW21 W, SW22 Z, SW23 L Alt, SW24 3, SW25 E, SW26 D, SW27 X, SW28 4, SW29 R, SW3 F3, SW30 F, SW31 C, SW32 5, SW33 T, SW34 G, SW35 V, SW36 6, SW37 Y, SW38 H, SW39 B, SW4 F2, SW40 Space, SW41 7, SW42 U, SW43 J, SW44 N, SW45 8, SW46 I, SW47 K, SW48 M, SW49 9, SW5 F4, SW50 O, SW51 L, SW52 ,, SW53 AltGr, SW54 ;, SW55 FN, SW56 0, SW57 P, SW58 ., SW59 R Ctrl, SW6 F5, SW60 -, SW61 [, SW62 ', SW63 /, SW64 =, SW65 ], SW66 RShift, SW67 Left, SW68 Back Space, SW69 \\, SW7 F7, SW70 Enter, SW71 UP, SW72 Down, SW73 Right, SW74 Num lock, SW75 7, SW76 1, SW77 4, SW78 /, SW79 8, SW8 F9, SW80 2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

Commit message: switches placed
Parts:
- added D90: 1N4148W, Diode_SMD:D_SOD-123, symbol Device:D_Small
- added SW91: Caps, acheron_MX:MX175, symbol acheronSymbols:MXSwitch
- SW40: footprint acheron_MX:MX625H -> acheron_MX:MX625
- SW63: footprint acheron_MX:MX150 -> acheron_MX:MX100
- SW69: footprint acheron_MX:MX100 -> acheron_MX:MX150
- SW75: value 7 -> N7
- SW76: value 1 -> N1
- SW77: value 4 -> N4
- SW78: value / -> N/
- SW79: value 8 -> N8
- SW80: value 2 -> N2
- SW81: value 5 -> N5
- SW82: value 0 -> N0
- SW83: value * -> N*
- SW84: value 9 -> N9
- SW85: value 3 -> N3
- SW86: value 6 -> N6
- SW87: value . -> N.
- SW88: value - -> N-
- SW89: value + -> N+
- SW90: value Enter -> PEenter
Connections:
- net COL3: now also SW91.1 (Col)
- net ROW3: now also D90.1 (K)
- new net: D90.2 (A), SW91.2 (Row)
Changed lines of the file:
@@
 F 0 "SW69" H 15750 8200 50  0000 L CNN
 F 1 "\\" H 15750 8100 79  0000 L CNN
-F 2 "acheron_MX:MX100" H 15850 8150 50  0001 C CNN
+F 2 "acheron_MX:MX150" H 15850 8150 50  0001 C CNN
 F 3 "" H 15850 8150 50  0001 C CNN
 	1    15850 8150
@@
 P 18050 7050
 F 0 "SW78" H 17950 7100 50  0000 L CNN
-F 1 "/" H 17950 7000 79  0000 L CNN
+F 1 "N/" H 17950 7000 79  0000 L CNN
 F 2 "acheron_MX:MX100" H 18050 7050 50  0001 C CNN
 F 3 "" H 18050 7050 50  0001 C CNN
@@
 P 17200 8150
 F 0 "SW75" H 17100 8200 50  0000 L CNN
-F 1 "7" H 17100 8100 79  0000 L CNN
+F 1 "N7" H 17100 8100 79  0000 L CNN
 F 2 "acheron_MX:MX100" H 17200 8150 50  0001 C CNN
 F 3 "" H 17200 8150 50  0001 C CNN
@@
 P 18050 8150
 F 0 "SW79" H 17950 8200 50  0000 L CNN
-F 1 "8" H 17950 8100 79  0000 L CNN
+F 1 "N8" H 17950 8100 79  0000 L CNN
 F 2 "acheron_MX:MX100" H 18050 8150 50  0001 C CNN
 F 3 "" H 18050 8150 50  0001 C CNN
@@
 P 18900 7050
 F 0 "SW83" H 18800 7100 50  0000 L CNN
-F 1 "*" H 18800 7000 79  0000 L CNN
+F 1 "N*" H 18800 7000 79  0000 L CNN
 F 2 "acheron_MX:MX100" H 18900 7050 50  0001 C CNN
 F 3 "" H 18900 7050 50  0001 C CNN
@@
 P 19750 7050
 F 0 "SW88" H 19650 7100 50  0000 L CNN
-F 1 "-" H 19650 7000 79  0000 L CNN
+F 1 "N-" H 19650 7000 79  0000 L CNN
 F 2 "acheron_MX:MX100" H 19750 7050 50  0001 C CNN
 F 3 "" H 19750 7050 50  0001 C CNN
@@
 P 18900 8150
 F 0 "SW84" H 18800 8200 50  0000 L CNN
-F 1 "9" H 18800 8100 79  0000 L CNN
+F 1 "N9" H 18800 8100 79  0000 L CNN
 F 2 "acheron_MX:MX100" H 18900 8150 50  0001 C CNN
 F 3 "" H 18900 8150 50  0001 C CNN
@@
 P 19750 8150
 F 0 "SW89" H 19650 8200 50  0000 L CNN
-F 1 "+" H 19650 8100 79  0000 L CNN
+F 1 "N+" H 19650 8100 79  0000 L CNN
 F 2 "acheron_MX:MX200V" H 19750 8150 50  0001 C CNN
 F 3 "" H 19750 8150 50  0001 C CNN
@@
 F 0 "SW63" H 14000 10350 50  0000 L CNN
 F 1 "/" H 14000 10250 79  0000 L CNN
-F 2 "acheron_MX:MX150" H 14100 10300 50  0001 C CNN
+F 2 "acheron_MX:MX100" H 14100 10300 50  0001 C CNN
 F 3 "" H 14100 10300 50  0001 C CNN
 	1    14100 10300
@@
 P 17250 9250
 F 0 "SW77" H 17150 9300 50  0000 L CNN
-F 1 "4" H 17150 9200 79  0000 L CNN
+F 1 "N4" H 17150 9200 79  0000 L CNN
 F 2 "acheron_MX:MX100" H 17250 9250 50  0001 C CNN
 F 3 "" H 17250 9250 50  0001 C CNN
@@
 P 18100 9250
 F 0 "SW81" H 18000 9300 50  0000 L CNN
-F 1 "5" H 18000 9200 79  0000 L CNN
+F 1 "N5" H 18000 9200 79  0000 L CNN
 F 2 "acheron_MX:MX100" H 18100 9250 50  0001 C CNN
 F 3 "" H 18100 9250 50  0001 C CNN
@@
 P 18950 9250
 F 0 "SW86" H 18850 9300 50  0000 L CNN
-F 1 "6" H 18850 9200 79  0000 L CNN
+F 1 "N6" H 18850 9200 79  0000 L CNN
 F 2 "acheron_MX:MX100" H 18950 9250 50  0001 C CNN
 F 3 "" H 18950 9250 50  0001 C CNN
@@
 P 19800 10300
 F 0 "SW90" H 19700 10350 50  0000 L CNN
-F 1 "Enter" H 19700 10250 79  0000 L CNN
+F 1 "PEenter" H 19700 10250 79  0000 L CNN
 F 2 "acheron_MX:MX200V" H 19800 10300 50  0001 C CNN
 F 3 "" H 19800 10300 50  0001 C CNN
@@
 P 17200 10300
 F 0 "SW76" H 17100 10350 50  0000 L CNN
-F 1 "1" H 17100 10250 79  0000 L CNN
+F 1 "N1" H 17100 10250 79  0000 L CNN
 F 2 "acheron_MX:MX100" H 17200 10300 50  0001 C CNN
 F 3 "" H 17200 10300 50  0001 C CNN
@@
 P 18050 10300
 F 0 "SW80" H 17950 10350 50  0000 L CNN
-F 1 "2" H 17950 10250 79  0000 L CNN
+F 1 "N2" H 17950 10250 79  0000 L CNN
 F 2 "acheron_MX:MX100" H 18050 10300 50  0001 C CNN
 F 3 "" H 18050 10300 50  0001 C CNN
@@
 P 18900 10300
 F 0 "SW85" H 18800 10350 50  0000 L CNN
-F 1 "3" H 18800 10250 79  0000 L CNN
+F 1 "N3" H 18800 10250 79  0000 L CNN
 F 2 "acheron_MX:MX100" H 18900 10300 50  0001 C CNN
 F 3 "" H 18900 10300 50  0001 C CNN
@@
 Connection ~ 4600 10700
 Wire Wire Line
-	4150 8150 4150 10300
+	4150 8150 4150 9200
 Connection ~ 3650 9600
 Connection ~ 6750 8150
@@
 	13150 8550 14100 8550
 Wire Wire Line
-	3650 8550 5450 8550
+	3650 8550 4600 8550
 Connection ~ 5900 8150
 Connection ~ 5900 9200
@@
 P 18100 11400
 F 0 "SW82" H 18000 11450 50  0000 L CNN
-F 1 "0" H 18000 11350 79  0000 L CNN
+F 1 "N0" H 18000 11350 79  0000 L CNN
 F 2 "acheron_MX:MX100" H 18100 11400 50  0001 C CNN
 F 3 "" H 18100 11400 50  0001 C CNN
@@
 P 18950 11400
 F 0 "SW87" H 18850 11450 50  0000 L CNN
-F 1 "." H 18850 11350 79  0000 L CNN
+F 1 "N." H 18850 11350 79  0000 L CNN
 F 2 "acheron_MX:MX100" H 18950 11400 50  0001 C CNN
 F 3 "" H 18950 11400 50  0001 C CNN
@@
 F 0 "SW40" H 9650 11450 50  0000 L CNN
 F 1 "Space" H 9600 11350 79  0000 L CNN
-F 2 "acheron_MX:MX625H" H 9750 11400 50  0001 C CNN
+F 2 "acheron_MX:MX625" H 9750 11400 50  0001 C CNN
 F 3 "" H 9750 11400 50  0001 C CNN
 	1    9750 11400
@@
 Wire Wire Line
 	12300 10700 13200 10700
+$Comp
+L Device:D_Small D90
+U 1 1 5D9B7DE0
+P 4600 8750
+F 0 "D90" V 4554 8818 50  0000 L CNN
+F 1 "1N4148W" V 4645 8818 50  0000 L CNN
+F 2 "Diode_SMD:D_SOD-123" V 4600 8750 50  0001 C CNN
+F 3 "~" V 4600 8750 50  0001 C CNN
+	1    4600 8750
+	0    1    1    0
+$EndComp
+$Comp
+L acheronSymbols:MXSwitch SW91
+U 1 1 5D9B7DE6
+P 4600 9200
+F 0 "SW91" H 4500 9250 50  0000 L CNN
+F 1 "Caps" H 4500 9150 79  0000 L CNN
+F 2 "acheron_MX:MX175" H 4600 9200 50  0001 C CNN
+F 3 "" H 4600 9200 50  0001 C CNN
+	1    4600 9200
+	1    0    0    -1
+$EndComp
+Wire Wire Line
+	4600 8650 4600 8550
+Connection ~ 4600 8550
+Wire Wire Line
+	4600 8550 5450 8550
+Wire Wire Line
+	4250 9200 4150 9200
+Connection ~ 4150 9200
+Wire Wire Line
+	4150 9200 4150 10300
 $EndSCHEMATC

Commit message: Routing
Connections:
- net COL1: now also U1.25 (PD4)
- net COL10: now also U1.37 (PF6)
- net COL11: now also U1.38 (PF5)
- net COL12: now also U1.39 (PF4)
- net COL13: now also SW54.1 (Col), SW55.1 (Col), SW58.1 (Col), U1.40 (PF1)
- net COL14: now also U1.41 (PF0)
- net COL2: now also U1.26 (PD6)
- net COL3: now also U1.27 (PD7)
- net COL4: now also U1.28 (PB4)
- net COL5: now also U1.29 (PB5)
- net COL6: now also U1.30 (PB6)
- net COL7: now also U1.31 (PC6)
- net COL8: now also U1.32 (PC7)
- net COL9: now also U1.36 (PF7)
Changed lines of the file:
@@
 Wire Wire Line
 	4150 9200 4150 10300
+Wire Wire Line
+	12700 8150 12800 8150
+Connection ~ 12800 8150
+Text GLabel 9000 2200 2    50   Input ~ 0
+COL8
+Text GLabel 9000 2100 2    50   Input ~ 0
+COL7
+Text GLabel 9000 1800 2    50   Input ~ 0
+COL6
+Text GLabel 9000 1700 2    50   Input ~ 0
+COL5
+Text GLabel 9000 1600 2    50   Input ~ 0
+COL4
+Text GLabel 9000 3100 2    50   Input ~ 0
+COL3
+Text GLabel 9000 3000 2    50   Input ~ 0
+COL2
+Text GLabel 9000 2800 2    50   Input ~ 0
+COL1
+Text GLabel 9000 4100 2    50   Input ~ 0
+COL9
+Text GLabel 9000 4000 2    50   Input ~ 0
+COL10
+Text GLabel 9000 3900 2    50   Input ~ 0
+COL11
+Text GLabel 9000 3800 2    50   Input ~ 0
+COL12
+Text GLabel 9000 3700 2    50   Input ~ 0
+COL13
+Text GLabel 9000 3600 2    50   Input ~ 0
+COL14
 $EndSCHEMATC
