File: Keyboard PCB/MA-65.kicad_pcb (KiCad board)
At the start: 2 copper layers, 151 parts, among them J1 USB_B_Mini, SW1 SW_Push, SW12 ESC, SW13 Tab, SW14 L Shift, SW15 L Ctrl, SW16 1, SW17 Q, SW18 A, SW19 S, SW2 `, SW20 2, SW21 W, SW22 Z, SW23 L Alt, SW24 3, SW25 E, SW26 D, SW27 X, SW28 4, SW29 R, SW3 PgUp, SW30 F, SW31 C, SW32 5, SW33 T, SW34 G, SW35 V, SW36 6, SW37 Y, SW38 H, SW39 B, SW4 PgDown, SW40 Space, SW41 7, SW42 U, SW43 J, SW44 N, SW45 8, SW46 I, SW47 K, SW48 M, SW49 9, SW5 Fn, SW50 O, SW51 L, SW52 ,, SW53 AltGr, SW54 ;, SW56 0, SW57 P, SW58 ., SW59 R Ctrl, SW6 Right, SW60 -, SW61 [, SW62 ', SW63 /, SW64 =, SW65 ], SW66 RShift, SW67 Left, SW68 Back Space, SW69 \, SW7 Back Space 2u, SW70 Enter, SW71 UP, SW72 Down, SW91 Caps, U1 ATmega32U4-AU, Y1 16mhz

Commit message: PCB Ma-65
Parts:
- added D10: 1N4148W, Diode_SMD:D_SOD-123, F.Cu at (89.2, -103.6)
- added D8: 1N4148W, Diode_SMD:D_SOD-123, F.Cu at (185.7, -112.7)
- added D9: 1N4148W, Diode_SMD:D_SOD-123, F.Cu at (319.1, -111.9)
- added SW11: PgUp, acheron_MX:MX100, F.Cu at (326.2, -111.9)
- added SW55: Win, acheron_MX:MX125, F.Cu at (66.7, -35.7)
- SW2: value ` -> Del
- SW3: value PgUp -> PgDn
- SW4: value PgDown -> Insert
- SW5: value Fn -> Fn2
- moved R3 323.2 mm to (168.2, -104.8), turned to 180 degrees
- moved SW54 313.2 mm to (245.3, -73.8)
- moved SW60 300.9 mm to (250.0, -111.9)
- moved SW70 278.5 mm to (295.3, -73.8)
- moved SW6 256.1 mm to (326.2, -35.7)
- moved SW53 254.8 mm to (233.4, -35.7)
- moved SW43 252.5 mm to (188.1, -73.8)
- moved SW47 250.6 mm to (207.2, -73.8)
- moved SW39 248.3 mm to (159.5, -54.8)
- moved SW35 242.9 mm to (140.5, -54.8)
- moved SW22 242.1 mm to (83.3, -54.8)
- moved SW59 236.3 mm to (257.2, -35.7)
- moved SW72 228.5 mm to (307.2, -35.7)
- moved SW71 227.6 mm to (307.2, -54.8)
- moved SW52 225.5 mm to (216.7, -54.8)
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Connections:
- SW3 pad 1: COL15 -> COL16
- SW4 pad 1: COL15 -> COL16
- SW5 pad 1: COL15 -> COL16
- SW6 pad 1: COL15 -> COL16
- SW66 pad 1: COL13 -> COL14
- SW67 pad 1: COL13 -> COL14
- SW71 pad 1: COL14 -> COL15
- SW72 pad 1: COL14 -> COL15
Other:
- board outline added: 314.3 x 104.8 mm
